File: 8080_keypad.sch (KiCad schematic (older format))
At the start: 23 parts

Commit message: Working on keyboard.
Parts:
- removed C?: 473, symbol C
- removed C?: 103, symbol C
- removed R?: 10k, symbol R
- removed R? (x2): 10k, symbol R_Variable
- removed U?: NE555, symbol NE555
- removed U?: 74HCT4075, symbol 74HCT4075
- removed U?: 74LS595, symbol 74LS595
- added C?: 470, symbol C_Small
- added R? (x2): 10k, symbol R_Variable
- added U?: 2716, symbol 2716
- added U?: 74LS123, symbol 74LS123
Connections:
- net labels added: COL_A, COL_B, COL_C, COL_D, COL_E, COL_F, COL_G, COL_H, ROW_A, ROW_B, ROW_C, ROW_D, ROW_E, ROW_F, ROW_G, ROW_H
- net labels removed: 1kHz
- wire segments 129 -> 57
- no-connect marks 1 -> 2
Other:
- note added: "2704/2708/2716\nCHARACTER DECODER"
- note added: "KEY LATCH"
- note added: "KEYBOARD MATRIX\n& DRIVER"
- note added: "LATCH & INTERRUPT\nSINGLE SHOTS"
- note added: "MATRIX DECODER"
- note added: "SHIFT AND CONTROL BUTTONS"
- note removed: "TODO: 8-Bit Ring Counter"
- note removed: "TODO: Keyboard Matrix"
- moved on the sheet: C?, R?, SW?, U?, U?A
