File: 8080_parallel_ports.sch (KiCad schematic (older format))
At the start: 11 parts

Commit message: Working on keyboard.
Connections:
- net A_PB0: now reaches U?.18 (PB0)
- net A_PB1: now reaches U?.19 (PB1)
- net A_PB2: now reaches U?.20 (PB2)
- net A_PB3: now reaches U?.21 (PB3)
- net A_PB4: now reaches U?.22 (PB4)
- net A_PB5: now reaches U?.23 (PB5)
- net A_PB6: now reaches U?.24 (PB6)
- net A_PB7: now reaches U?.25 (PB7)
Other:
- note added: "KEYBOARD IN"
- note added: "KEYPAD"
- note added: "VIDEO"
Changed lines of the file:
@@
 $Descr A4 11693 8268
 encoding utf-8
-Sheet 4 7
+Sheet 4 9
 Title "8080 Single Board Computer"
 Date "2017-09-30"
@@
 Text GLabel 8800 1750 2    60   Input ~ 0
 A_PA7
+Text GLabel 8800 1950 2    60   Input ~ 0
+A_PB0
+Text GLabel 8800 2050 2    60   Input ~ 0
+A_PB1
+Text GLabel 8800 2150 2    60   Input ~ 0
+A_PB2
+Text GLabel 8800 2250 2    60   Input ~ 0
+A_PB3
+Text GLabel 8800 2350 2    60   Input ~ 0
+A_PB4
+Text GLabel 8800 2450 2    60   Input ~ 0
+A_PB5
+Text GLabel 8800 2550 2    60   Input ~ 0
+A_PB6
+Text GLabel 8800 2650 2    60   Input ~ 0
+A_PB7
+$Sheet
+S 4600 8350 3800 2500
+U 59D83EF6
+F0 "Video" 59
+F1 "8080_video.sch" 59
+$EndSheet
+Text Notes 2050 9550 0    118  ~ 0
+KEYPAD
+Text Notes 6300 9600 0    118  ~ 0
+VIDEO
+Text Notes 9350 1450 0    60   ~ 0
+KEYBOARD IN
 $EndSCHEMATC
